File: USB_Protect_A.sch (EAGLE design)
At the start: 6 parts, among them J1 61400416021, U1 SP3003-02JTG

Commit message: Update
Update details
Parts:
- removed LOGO2: OSHW-LOGOS, SparkFun-Aesthetics:OSHW-LOGOS
- removed U$1: XDESIG5MM, xdesig:XDESIG5MM
- added LOGO1: OSHW-LOGOS, Echidna_shield_LBR:OSHW-LOGOS
Changed lines of the file:
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@@
 <part name="U1" library="SP3003-02JTG" deviceset="SP3003-02JTG" device=""/>
 <part name="J1" library="USB_female" deviceset="61400416021" device=""/>
-<part name="LOGO2" library="SparkFun-Aesthetics" deviceset="OSHW-LOGO" device="S"/>
-<part name="U$1" library="xdesig" deviceset="XDESIG" device="5MM"/>
+<part name="LOGO1" library="Echidna_shield_LBR" deviceset="OSHW-LOGO" device="S"/>
 </parts>
 <sheets>
@@
                            IEC61000-4-2 (Air) ±15 kV</text>
 <text x="213.36" y="17.78" size="2.54" layer="97"> 1A / 12V</text>
-<text x="165.1" y="27.94" size="1.6764" layer="97" font="vector">Attribution-ShareAlike 4.0 International (CC BY-SA 4.0) by XDeSIG</text>
+<text x="165.1" y="27.94" size="2.54" layer="97">Attribution-ShareAlike 4.0 International (CC BY-SA 4.0) by XDeSIG</text>
 <text x="256.54" y="7.62" size="2.54" layer="97">001</text>
 </plain>
@@
 <instance part="U1" gate="A" x="121.92" y="88.9"/>
 <instance part="J1" gate="G$1" x="165.1" y="116.84" rot="MR180"/>
-<instance part="LOGO2" gate="G$1" x="251.46" y="48.26"/>
-<instance part="U$1" gate="G$1" x="256.54" y="27.94"/>
+<instance part="LOGO1" gate="G$1" x="124.46" y="20.32"/>
 </instances>
 <busses>
@@
 </sheet>
 </sheets>
+<errors>
+</errors>
 </schematic>
 </drawing>
